File: buck/buck.kicad_pcb (KiCad board)
At the start: 2 copper layers, 37.8 x 17.8 mm, 15 parts, among them IC1 TPS630702RNMR

Commit message: made prod file
Other:
- board size 37.8 x 17.8 mm -> 13.6 x 11.2 mm
Changed lines of the file:
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@@
-	)
-	(gr_rect
-		(start 176.4 63.4)
-		(end 197.4 81.2)
-		(stroke
-			(width 0.05)
-			(type default)
-		)
-		(fill no)
-		(layer "Edge.Cuts")
 	)
 	(gr_rect
